File: eagle/current_sensor_pcb/current_sensor.sch (EAGLE design)
At the start: 1 part, among them M1 ARDUINO-NANO-LONG

Commit message: pcb design ready
Parts:
- added J1, J2, J3, J4, J5, J6: (no value), SparkFun-Connectors:CONN_02LOCK_LONGPADS
- added R1, R2: (no value), SparkFun-Resistors:RESISTORAXIAL-0.3
- added U$1: CURRENT-SENSOR-ACS712, diy-modules:CURRENT-SENSOR-ACS712
- added X1, X2, X3: MST2V, con-phoenix-508:MST2V
Connections:
- new net 3V3: J3.1, M1.3V3
- new net 5V: J2.1, M1.5V
- new net A2: J4.1, M1.A2
- new net A3: J4.2, M1.A3
- new net D5: J5.1, M1.D5
- new net D6: J5.2, M1.D6
- new net GND: J1.2, J2.2, J3.2, J6.2, M1.GND.2, R2.1, U$1.GND, X1-2.1, X2-2.1
- new net N$1: M1.A0, U$1.OUT
- new net N$2: R1.2, X1-1.1, X3-2.1
- new net N$3: J1.1, U$1.VCC
- new net N$5: M1.A1, R1.1, R2.2
- new net N$6: X2-1.1, X3-1.1
- new net VIN: J6.1, M1.VIN
Other:
- moved on the sheet: M1
